File: hardware/RocketTracker/RocketTracker/_autosave-LiPoPowerSimple.kicad_sch (KiCad schematic)
At the start: 35 parts, among them J201 LiPo, SW201 Power Switch, U201 MCP73871-1CC, U202 TPS63070RNMR

Commit message: ガーバー出力
Changed lines of the file:
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@@
 		(on_board yes)
 		(dnp no)
-		(fields_autoplaced yes)
 		(property "Reference" "R211"
-			(at 208.28 58.42 90)
+			(at 208.28 60.96 90)
 			(effects
 				(font
@@
 		)
 		(property "Value" "100k"
-			(at 208.28 60.96 90)
+			(at 208.28 62.738 90)
 			(effects
 				(font
@@
 		(dnp no)
 		(property "Reference" "R204"
-			(at 68.58 115.57 0)
-			(effects
-				(font
+			(at 69.85 115.57 0)
+			(effects
+				(font
