File: hardware/RocketTracker/RocketTracker/RocketTracker.kicad_sch (KiCad schematic)
At the start: 4 parts, among them Q201 AO3400A

Commit message: シルク入れた
Parts:
- added B101: ~, WOBCLibrary:Board_1U_60x60, symbol WOBCLibrary:Board
- added R103, R104: 10k, Resistor_SMD:R_0402_1005Metric, symbol Device:R
- renumbered BZ201 to BZ101, Q201 to Q101, R107 to R101, R104 to R102
Connections:
- net ESP32C3core/IO1: now also R103.1, R104.2
- net GND: now also B101.GND, R104.1
- new net VPP: R103.2
- no-connect marks 0 -> 5
Other:
- sheet ESP32C3core: file untitled.kicad_sch -> ESP32C3core.kicad_sch

Commit message: コンデンサ，ダイオード追加
Parts:
- removed R104: 10k, Resistor_SMD:R_0402_1005Metric, symbol Device:R
- added C211: 22uF, Capacitor_SMD:C_0805_2012Metric, symbol Device:C
- added D201: D, Diode_SMD:D_SOD-323, symbol Device:D
- added R203: 100k, Resistor_SMD:R_0402_1005Metric, symbol Device:R
- R103: value 10k -> 100k; LCSC C25744 -> C25741
Connections:
- net ESP32C3core/IO1: now also R203.2
- net ESP32C3core/IO10: no longer R102.1
- net GND: now also C211.2, R203.1
- net at BZ101.2 (-), Q101.3 (D): now also D201.2 (A)
- net at Q101.1 (G), R101.1: now also R102.1
- net VDD renamed LiPo/MCPOUT
- net LiPo/MCPOUT: now also C211.1, D201.1 (K)
Other:
- sheet LiPo ports: added MCPOUT; removed none
- moved on the sheet: BZ101, R101, R102
